Commit message: gazebo additions

File: simple2wheeler/urdf/simple2wheeler.xacro (robot description, xacro)
@@ -91,3 +91,54 @@
         <joint_properties damping="1.0" friction="1.0"/>
     </joint>
+    <link name="camera_link">
+        <collision>
+        </collision>
+        <visual>
+        </visual>
+    </link>
+    <joint name="camera_joint" type="fixed">
+        <origin rpy="0 0 0" xyz="0.25 0.07 0.07"/>
+        <child link="camera_link"/>
+        <parent link="link_chassis"/>
+    </joint>
+    <!-- gazebo ros plugin kameralle -->
+    <gazebo reference="camera_link">
+        <sensor type="camera" name="camera_sensor">
+            <update_rate>30.0</update_rate>
+            <camera>
+                <horizontal_fov>1.34</horizontal_fov>
+                <image>
+                    <format>R8G8B8</format>
+                    <width>320</width>
+                    <height>240</height>
+                </image>
+                <clip>
+                    <near>0.01</near>
+                    <far>30</far>
+                </clip>
+            </camera>
+            <plugin name="camera_controller" filename="libgazebo_ros_camera.so">
+                <updateRate>30.0</updateRate>
+                <cameraName>/camera</cameraName>
+                <imageTopicName>image_raw</imageTopicName>
+                <cameraInfoTopicName>camera_info</cameraInfoTopicName>
+                <frameName>camera_link</frameName>
+                <hackBaseline>0.07</hackBaseline>
+            </plugin>
+        </sensor>
+    </gazebo>
+    <!-- gazebo ros plugin robotin liikuttamiseksi -->
+    <gazebo>
+        <plugin filename="libgazebo_ros_diff_drive.so" name="differential_drive_controller">
+            <leftJoint>joint_left_wheel</leftJoint>
+            <rightJoint>joint_right_wheel</rightJoint>
+            <wheelSeparation>0.2</wheelSeparation>
+            <wheelDiameter>0.2</wheelDiameter>
+            <torque>0.1</torque>
+            <commandTopic>cmd_vel</commandTopic>
+            <odometryTopic>odom</odometryTopic>
+            <odometryFrame>odom</odometryFrame>
+            <robotBaseFrame>base_link</robotBaseFrame>
+        </plugin>
+    </gazebo>
 </robot>

Commit message: Random roaming in arena

File: simple2wheeler/urdf/simple2wheeler.xacro (robot description, xacro)
@@ -40,29 +40,4 @@
         </visual>
     </link>
-    <link name="link_right_wheel">
-        <inertial>
-            <mass value="0.2"/>
-            <inertia ixx="0.0005266" ixy="0" ixz="0"
-                     iyy="0.0005266"  iyz="0" izz="0.001"
-        /></inertial>
-        <collision name="collision_link_right_wheel">
-            <geometry>
-                <cylinder length="0.04" radius="0.1"/>
-            </geometry>
-        </collision>
-        <visual name ="visual_right_wheel">
-            <geometry>
-                <cylinder length="0.04" radius="0.1"/>
-            </geometry>
-        </visual>
-    </link>
-    <joint name="joint_right_wheel" type="continuous">
-        <origin rpy="1.5707 0 0" xyz="-0.05 0.15 0"/>
-        <child link="link_right_wheel"/>
-        <parent link="link_chassis"/>
-        <axis rpy="0 0 0" xyz="0 0 1"/>
-        <limit effort="10" velocity="10"/>
-        <joint_properties damping="1.0" friction="1.0"/>
-    </joint>
     <link name="link_left_wheel">
         <inertial>
@@ -85,4 +60,29 @@
         <origin rpy="1.5707 0 0" xyz="-0.05 -0.15 0"/>
         <child link="link_left_wheel"/>
+        <parent link="link_chassis"/>
+        <axis rpy="0 0 0" xyz="0 0 1"/>
+        <limit effort="10" velocity="10"/>
+        <joint_properties damping="1.0" friction="1.0"/>
+    </joint>
+    <link name="link_right_wheel">
+        <inertial>
+            <mass value="0.2"/>
+            <inertia ixx="0.0005266" ixy="0" ixz="0"
+                     iyy="0.0005266"  iyz="0" izz="0.001"
+        /></inertial>
+        <collision name="collision_link_right_wheel">
+            <geometry>
+                <cylinder length="0.04" radius="0.1"/>
+            </geometry>
+        </collision>
+        <visual name ="visual_right_wheel">
+            <geometry>
+                <cylinder length="0.04" radius="0.1"/>
+            </geometry>
+        </visual>
+    </link>
+    <joint name="joint_right_wheel" type="continuous">
+        <origin rpy="1.5707 0 0" xyz="-0.05 0.15 0"/>
+        <!--child link="link_left_wheel"/-->
         <child link="link_right_wheel"/>
         <parent link="link_chassis"/>
